File: ir_read_mod.sch (KiCad schematic (older format))
At the start: 21 parts, among them J1 Conn_01x04_Female, J2 Conn_01x05_Female, J3 Conn_01x01_Female, J4 Conn_01x02_Female, Q1 Q_Photo_NPN, SW1 SW_Coded_SH-7070, SW2 SW_SPDT, U1 PIC16F1503-IP

Commit message: Update: fix parts
Parts:
- removed D2: LED, LED_THT:LED_D5.0mm, symbol Device:LED
- removed J3: Conn_01x01_Female, Connector_PinSocket_2.54mm:PinSocket_1x01_P2.54mm_Vertical, symbol Connector:Conn_01x01_Female
- removed J4: Conn_01x02_Female, Connector_PinSocket_2.54mm:PinSocket_1x02_P2.54mm_Vertical, symbol Connector:Conn_01x02_Female
- added R10, R11, R8, R9: 300, Resistor_SMD:R_0603_1608Metric_Pad1.05x0.95mm_HandSolder, symbol Device:R
- D1: footprint LED_THT:LED_D5.0mm -> LED_SMD:LED_0603_1608Metric_Castellated
- D2: renamed from D3; footprint LED_THT:LED_D5.0mm -> LED_SMD:LED_0603_1608Metric_Castellated
- D3: renamed from D4; footprint LED_THT:LED_D5.0mm -> LED_SMD:LED_0603_1608Metric_Castellated
- D4: renamed from D5; footprint LED_THT:LED_D5.0mm -> LED_SMD:LED_0603_1608Metric_Castellated
- R1: renamed from R3; footprint Resistor_THT:R_Axial_DIN0207_L6.3mm_D2.5mm_P7.62mm_Horizontal -> Resistor_SMD:R_0805_2012Metric_Pad1.15x1.40mm_HandSolder
- R2: renamed from R4; footprint Resistor_THT:R_Axial_DIN0207_L6.3mm_D2.5mm_P7.62mm_Horizontal -> Resistor_SMD:R_0805_2012Metric_Pad1.15x1.40mm_HandSolder
- R3: renamed from R5; footprint Resistor_THT:R_Axial_DIN0207_L6.3mm_D2.5mm_P7.62mm_Horizontal -> Resistor_SMD:R_0805_2012Metric_Pad1.15x1.40mm_HandSolder
- R4: renamed from R6; footprint Resistor_THT:R_Axial_DIN0207_L6.3mm_D2.5mm_P7.62mm_Horizontal -> Resistor_SMD:R_0805_2012Metric_Pad1.15x1.40mm_HandSolder
- R5: renamed from R7; footprint Resistor_THT:R_Axial_DIN0207_L6.3mm_D2.5mm_P7.62mm_Horizontal -> Resistor_SMD:R_0805_2012Metric_Pad1.15x1.40mm_HandSolder
- R6: renamed from R1; footprint Resistor_THT:R_Axial_DIN0207_L6.3mm_D2.5mm_P7.62mm_Horizontal -> Resistor_SMD:R_0805_2012Metric_Pad1.15x1.40mm_HandSolder
- R7: renamed from R2; footprint Resistor_THT:R_Axial_DIN0207_L6.3mm_D2.5mm_P7.62mm_Horizontal -> Resistor_SMD:R_0805_2012Metric_Pad1.15x1.40mm_HandSolder
- renumbered J1 to J3
Connections:
- wire segments 103 -> 98
